Commit message: new version

File: SAR_ROS_packages/sar_simulations/urdf/my_camera.urdf.xacro (robot description, xacro)
@@ -36,10 +36,10 @@
       <gazebo reference="camera_link">
         <sensor type="camera" name="camera1">
-          <update_rate>30.0</update_rate>
+          <update_rate>20</update_rate>
           <camera name="head">
         <horizontal_fov>1.3962634</horizontal_fov>
         <image>
-          <width>640</width>
-          <height>480</height>
+          <width>800</width>
+          <height>800</height>
           <format>R8G8B8</format>
         </image>
@@ -59,5 +59,5 @@
           <plugin name="camera_controller" filename="libgazebo_ros_camera.so">
         <alwaysOn>true</alwaysOn>
-        <updateRate>0.0</updateRate>
+        <updateRate>20</updateRate>
         <cameraName>camera1</cameraName>
         <imageTopicName>image_raw</imageTopicName>

File: SAR_ROS_packages/sar_simulations/urdf/nexus_own.xacro (robot description, xacro)
@@ -1,119 +1,123 @@
 <?xml version="1.0"?>
 <robot name="nexus_4wd_mecanum" xmlns:xacro="http://ros.org/wiki/xacro">
-	  <xacro:include filename="$(find nexus_4wd_mecanum_description)/urdf/nexus_4wd_mecanum.xacro" />
-	  <xacro:property name="camera_link" value="0.05" />
+	<xacro:include filename="$(find nexus_4wd_mecanum_description)/urdf/nexus_4wd_mecanum.xacro" />
+	<xacro:property name="camera_link" value="0.05" />
 	<!-- height of link_7 is 0.03 -->
-	  <joint name="camera_joint" type="fixed">
-	    <!-- <axis xyz="0 0 0" /> -->
-	    <origin xyz="0 0 0.2" rpy="0 0 0"/>
-	    <parent link="base_link"/>
-	    <child link="camera_link"/>
-	  </joint>
-	  <!-- Camera -->
-	  <link name="camera_link">
-	    <collision>
-	      <origin xyz="0 0 0.2" rpy="0 0 0"/>
-	      <geometry>
-		 <box size="1 ${camera_link} 0.025"/>
-	      </geometry>
-	    </collision>
-	    <visual>
-	      <origin xyz="0 0 0" rpy="0 0 0"/>
-	      <geometry>
-		 <box size="${camera_link} ${camera_link} 0.025"/>
-	      </geometry>
-	      <material name="red"/>
-	    </visual>
-	    <inertial>
-	      <mass value="1e-5" />
-	      <origin xyz="0 0 0" rpy="0 0 0"/>
-	      <inertia ixx="1e-6" ixy="0" ixz="0" iyy="1e-6" iyz="0" izz="1e-6" />
-	    </inertial>
-	  </link>
-	  <joint name="imu_sensor_joint" type="fixed">
-		<axis xyz="0 0 1" />
-		<origin xyz="0.0 0.0 0.0" rpy="0 0 0"/>
-		<parent link="base_link"/>
-		<child link="imu_sensor_link"/>
-    	  </joint>
-     	  <link name="imu_sensor_link">
+	<joint name="camera_joint" type="fixed">
+		<!-- <axis xyz="0 0 0" /> -->
+		<origin xyz="0 0 0.2" rpy="0 0 0" />
+		<parent link="base_link" />
+		<child link="camera_link" />
+	</joint>
+	<!-- Camera -->
+	<link name="camera_link">
 		<collision>
-		    <origin xyz="0 0 0" rpy="0 0 0"/>
-		    <geometry>
-		        <box size="0.02 0.02 0.02"/>
-		    </geometry>
+			<origin xyz="0 0 0.2" rpy="0 0 0" />
+			<geometry>
+				<box size="1 ${camera_link} 0.025" />
+			</geometry>
 		</collision>
 		<visual>
-		    <origin xyz="0 0 0" rpy="0 0 0"/>
-		    <geometry>
-		        <box size="0.02 0.02 0.02"/>
-		    </geometry>
-		    <material name="iRobot/Red"/>
+			<origin xyz="0 0 0" rpy="0 0 0" />
+			<geometry>
+				<box size="${camera_link} ${camera_link} 0.025" />
+			</geometry>
+			<material name="red" />
 		</visual>
 		<inertial>
-		    <mass value="0.001" />
-		    <origin xyz="0 0 0" rpy="0 0 0"/>
-		    <inertia ixx="0.00000015" ixy="0" ixz="0" iyy="0.00000015" iyz="0" izz="0.00000015" />
+			<mass value="1e-5" />
+			<origin xyz="0 0 0" rpy="0 0 0" />
+			<inertia ixx="1e-6" ixy="0" ixz="0" iyy="1e-6" iyz="0" izz="1e-6" />
 		</inertial>
-    	  </link>
-    	  <gazebo reference="imu_sensor_link">
+	</link>
+	<joint name="imu_sensor_joint" type="fixed">
+		<axis xyz="0 0 1" />
+		<origin xyz="0.0 0.0 0.0" rpy="0 0 0" />
+		<parent link="base_link" />
+		<child link="imu_sensor_link" />
+	</joint>
+	<link name="imu_sensor_link">
+		<collision>
+			<origin xyz="0 0 0" rpy="0 0 0" />
+			<geometry>
+				<box size="0.02 0.02 0.02" />
+			</geometry>
+		</collision>
+		<visual>
+			<origin xyz="0 0 0" rpy="0 0 0" />
+			<geometry>
+				<box size="0.02 0.02 0.02" />
+			</geometry>
+			<material name="iRobot/Red" />
+		</visual>
+		<inertial>
+			<mass value="0.001" />
+			<origin xyz="0 0 0" rpy="0 0 0" />
+			<inertia ixx="0.00000015" ixy="0" ixz="0" iyy="0.00000015" iyz="0" izz="0.00000015" />
+		</inertial>
+	</link>
+	<gazebo reference="imu_sensor_link">
 		<gravity>true</gravity>
 		<sensor name='imu_sensor' type='imu'>
-		    <always_on>1</always_on>
-		    <update_rate>100</update_rate>
-		    <visualize>1</visualize>
-		    <topic>__default_topic__</topic>
-		    <plugin name='imu_plugin' filename='libgazebo_ros_imu_sensor.so'>
-		    	<robotNamespace>Mi_imu</robotNamespace>
-		        <topicName>imu_data</topicName>
-		        <bodyName>imu_sensor_link</bodyName>
-		        <updateRateHZ>10.0</updateRateHZ>
-		        <gaussianNoise>0.0</gaussianNoise>
-		        <xyzOffset>0 0 0</xyzOffset>
-		        <rpyOffset>0 0 0</rpyOffset>
-		        <frameName>imu_sensor_link</frameName>
-		    </plugin>
-		    <pose>0 0 0 0 0 0</pose>
+			<always_on>1</always_on>
+			<update_rate>100</update_rate>
+			<visualize>1</visualize>
+			<topic>__default_topic__</topic>
+			<plugin name='imu_plugin' filename='libgazebo_ros_imu_sensor.so'>
+				<robotNamespace></robotNamespace>
+				<topicName>imu</topicName>
+				<bodyName>imu_sensor_link</bodyName>
+				<updateRateHZ>10.0</updateRateHZ>
+				<gaussianNoise>0.0</gaussianNoise>
+				<xyzOffset>0 0 0</xyzOffset>
+				<rpyOffset>0 0 0</rpyOffset>
+				<frameName>imu_sensor_link</frameName>
+			</plugin>
+			<pose>0 0 0 0 0 0</pose>
 		</sensor>
-    	  </gazebo>
-	      <!-- camera -->
-	      <gazebo reference="camera_link">
-		<sensor type="camera" name="camera1">
-		  <update_rate>30.0</update_rate>
-		  <camera name="head">
-		<horizontal_fov>1.3962634</horizontal_fov>
-		<image>
-		  <width>800</width>
-		  <height>800</height>
-		  <format>R8G8B8</format>
-		</image>
-		<clip>
-		  <near>0.02</near>
-		  <far>300</far>
-		</clip>
-		<noise>
-		  <type>gaussian</type>
-		  <!-- Noise is sampled independently per pixel on each frame.
+	</gazebo>
+	<!-- camera -->
+	<gazebo reference="camera_link">
+		<sensor type="camera" name="camera">
+			<update_rate>30.0</update_rate>
+			<camera name="head">
+				<horizontal_fov>1.3962634</horizontal_fov>
+				<image>
+					<width>640</width>
+					<height>480</height>
+					<format>R8G8B8</format>
+				</image>
+				<clip>
+					<near>0.02</near>
+					<far>300</far>
+				</clip>
+				<noise>
+					<type>gaussian</type>
+					<!-- Noise is sampled independently per pixel on each frame.
 		       That pixel's noise value is added to each of its color
 		       channels, which at that point lie in the range [0,1]. -->
-		  <mean>0.0</mean>
-		  <stddev>0.007</stddev>
-		</noise>
-		  </camera>
-		  <plugin name="camera_controller" filename="libgazebo_ros_camera.so">
-		<alwaysOn>true</alwaysOn>
-		<updateRate>0.0</updateRate>
-		<cameraName>camera1</cameraName>
-		<imageTopicName>image_raw</imageTopicName>
-		<cameraInfoTopicName>camera_info</cameraInfoTopicName>
-		<frameName>camera_link</frameName>
-		<hackBaseline>0.07</hackBaseline>
-		<distortionK1>0.0</distortionK1>
-		<distortionK2>0.0</distortionK2>
-		<distortionK3>0.0</distortionK3>
-		<distortionT1>0.0</distortionT1>
-		<distortionT2>0.0</distortionT2>
-		  </plugin>
+					<mean>0.0</mean>
+					<stddev>0</stddev>
+				</noise>
+			</camera>
+			<plugin name="camera_controller" filename="libgazebo_ros_camera.so">
+				<alwaysOn>true</alwaysOn>
+				<updateRate>0.0</updateRate>
+				<cameraName>camera</cameraName>
+				<imageTopicName>image_raw</imageTopicName>
+				<cameraInfoTopicName>camera_info</cameraInfoTopicName>
+				<frameName>camera_link</frameName>
+				<hackBaseline>0.7</hackBaseline>
+				<distortionK1>0.0</distortionK1>
+				<distortionK2>0.0</distortionK2>
+				<distortionK3>0.0</distortionK3>
+				<distortionT1>0.0</distortionT1>
+				<distortionT2>0.0</distortionT2>
+				<CxPrime>0</CxPrime>
+				<Cx>0.0</Cx>
+				<Cy>0.0</Cy>
+				<focalLength>0.0</focalLength>
+			</plugin>
 		</sensor>
-	      </gazebo>
+	</gazebo>
 </robot>

Commit message: added lidar sensor

File: SAR_ROS_packages/sar_simulations/urdf/my_camera.urdf.xacro (robot description, xacro)
@@ -74,2 +74,3 @@
       </gazebo>
   </xacro:macro>
+</robot>

File: SAR_ROS_packages/sar_simulations/urdf/nexus_own.xacro (robot description, xacro)
@@ -57,4 +57,31 @@
 		</inertial>
 	</link>
+	<joint name="hokuyo_joint" type="fixed">
+		<axis xyz="0 1 0" />
+		<origin xyz="0 0 0.1" rpy="0 0 0"/>
+		<parent link="base_link"/>
+		<child link="hokuyo_link"/>
+	  </joint>
+	  <!-- Hokuyo Laser -->
+	  <link name="hokuyo_link">
+		<collision>
+		  <origin xyz="0 0 0" rpy="0 0 0"/>
+		  <geometry>
+		<box size="0.1 0.1 0.1"/>
+		  </geometry>
+		</collision>
+		<visual>
+			<origin xyz="0 0 0" rpy="0 0 0" />
+			<geometry>
+				<box size="${camera_link} ${camera_link} 0.025" />
+			</geometry>
+			<material name="red" />
+		</visual>
+		<inertial>
+		  <mass value="1e-5" />
+		  <origin xyz="0 0 0" rpy="0 0 0"/>
+		  <inertia ixx="1e-6" ixy="0" ixz="0" iyy="1e-6" iyz="0" izz="1e-6" />
+		</inertial>
+	  </link>
 	<gazebo reference="imu_sensor_link">
 		<gravity>true</gravity>
@@ -121,3 +148,38 @@
 		</sensor>
 	</gazebo>
+	<gazebo reference="hokuyo_link">
+		<sensor type="ray" name="head_hokuyo_sensor">
+		  <pose>0 0 0 0 0 0</pose>
+		  <visualize>true</visualize>
+		  <update_rate>40</update_rate>
+		  <ray>
+			<scan>
+			  <horizontal>
+				<samples>720</samples>
+				<resolution>1</resolution>
+				<min_angle>-1.570796</min_angle>
+				<max_angle>1.570796</max_angle>
+			  </horizontal>
+			</scan>
+			<range>
+			  <min>0.10</min>
+			  <max>30.0</max>
+			  <resolution>0.01</resolution>
+			</range>
+			<noise>
+			  <type>gaussian</type>
+			  <!-- Noise parameters based on published spec for Hokuyo laser
+				   achieving "+-30mm" accuracy at range < 10m.  A mean of 0.0m and
+				   stddev of 0.01m will put 99.7% of samples within 0.03m of the true
+				   reading. -->
+			  <mean>0.0</mean>
+			  <stddev>0.01</stddev>
+			</noise>
+		  </ray>
+		  <plugin name="gazebo_ros_head_hokuyo_controller" filename="libgazebo_ros_laser.so">
+			<topicName>/laser/scan</topicName>
+			<frameName>hokuyo_link</frameName>
+		  </plugin>
+		</sensor>
+	  </gazebo>
 </robot>
